Commit message: merging master into C_Iris

File: manipulation/models/jaco_description/urdf/j2s7s300.urdf (robot description, URDF)
Before this commit: robot j2s7s300, 16 links, 15 joints
Joints:
- joint j2s7s300_joint_1: limit lower=-174.532925 upper=174.532925 effort=2000 velocity=1 -> lower=-174.532925 upper=174.532925 effort=2000 velocity=0.63
- joint j2s7s300_joint_2: limit lower=0.523598775598 upper=5.75958653158 effort=2000 velocity=1 -> lower=0.523598775598 upper=5.75958653158 effort=2000 velocity=0.63
- joint j2s7s300_joint_3: limit lower=-174.532925 upper=174.532925 effort=2000 velocity=1 -> lower=-174.532925 upper=174.532925 effort=2000 velocity=0.63
- joint j2s7s300_joint_4: limit lower=0.523598775598 upper=5.75958653158 effort=2000 velocity=1 -> lower=0.523598775598 upper=5.75958653158 effort=2000 velocity=0.63
- joint j2s7s300_joint_5: limit lower=-174.532925 upper=174.532925 effort=2000 velocity=1 -> lower=-174.532925 upper=174.532925 effort=2000 velocity=0.85
- joint j2s7s300_joint_6: limit lower=0.523598775598 upper=5.75958653158 effort=2000 velocity=1 -> lower=0.523598775598 upper=5.75958653158 effort=2000 velocity=0.85
- joint j2s7s300_joint_7: limit lower=-174.532925 upper=174.532925 effort=2000 velocity=1 -> lower=-174.532925 upper=174.532925 effort=2000 velocity=0.85

File: manipulation/models/jaco_description/urdf/j2s7s300_arm.urdf (robot description, URDF)
Before this commit: robot j2s7s300_arm, 9 links, 8 joints
Joints:
- joint j2s7s300_joint_1: limit lower=-174.532925 upper=174.532925 effort=2000 velocity=1 -> lower=-174.532925 upper=174.532925 effort=2000 velocity=0.63
- joint j2s7s300_joint_2: limit lower=0.523598775598 upper=5.75958653158 effort=2000 velocity=1 -> lower=0.523598775598 upper=5.75958653158 effort=2000 velocity=0.63
- joint j2s7s300_joint_3: limit lower=-174.532925 upper=174.532925 effort=2000 velocity=1 -> lower=-174.532925 upper=174.532925 effort=2000 velocity=0.63
- joint j2s7s300_joint_4: limit lower=0.523598775598 upper=5.75958653158 effort=2000 velocity=1 -> lower=0.523598775598 upper=5.75958653158 effort=2000 velocity=0.63
- joint j2s7s300_joint_5: limit lower=-174.532925 upper=174.532925 effort=2000 velocity=1 -> lower=-174.532925 upper=174.532925 effort=2000 velocity=0.85
- joint j2s7s300_joint_6: limit lower=0.523598775598 upper=5.75958653158 effort=2000 velocity=1 -> lower=0.523598775598 upper=5.75958653158 effort=2000 velocity=0.85
- joint j2s7s300_joint_7: limit lower=-174.532925 upper=174.532925 effort=2000 velocity=1 -> lower=-174.532925 upper=174.532925 effort=2000 velocity=0.85

File: manipulation/models/jaco_description/urdf/j2s7s300_arm_sphere_collision.urdf (robot description, URDF)
Before this commit: robot j2s7s300_arm, 9 links, 8 joints
Joints:
- joint j2s7s300_joint_1: limit lower=-174.532925 upper=174.532925 effort=2000 velocity=1 -> lower=-174.532925 upper=174.532925 effort=2000 velocity=0.63
- joint j2s7s300_joint_2: limit lower=0.523598775598 upper=5.75958653158 effort=2000 velocity=1 -> lower=0.523598775598 upper=5.75958653158 effort=2000 velocity=0.63
- joint j2s7s300_joint_3: limit lower=-174.532925 upper=174.532925 effort=2000 velocity=1 -> lower=-174.532925 upper=174.532925 effort=2000 velocity=0.63
- joint j2s7s300_joint_4: limit lower=0.523598775598 upper=5.75958653158 effort=2000 velocity=1 -> lower=0.523598775598 upper=5.75958653158 effort=2000 velocity=0.63
- joint j2s7s300_joint_5: limit lower=-174.532925 upper=174.532925 effort=2000 velocity=1 -> lower=-174.532925 upper=174.532925 effort=2000 velocity=0.85
- joint j2s7s300_joint_6: limit lower=0.523598775598 upper=5.75958653158 effort=2000 velocity=1 -> lower=0.523598775598 upper=5.75958653158 effort=2000 velocity=0.85
- joint j2s7s300_joint_7: limit lower=-174.532925 upper=174.532925 effort=2000 velocity=1 -> lower=-174.532925 upper=174.532925 effort=2000 velocity=0.85

File: manipulation/models/jaco_description/urdf/j2s7s300_sphere_collision.urdf (robot description, URDF)
Before this commit: robot j2s7s300, 16 links, 15 joints
Joints:
- joint j2s7s300_joint_1: limit lower=-174.532925 upper=174.532925 effort=2000 velocity=1 -> lower=-174.532925 upper=174.532925 effort=2000 velocity=0.63
- joint j2s7s300_joint_2: limit lower=0.523598775598 upper=5.75958653158 effort=2000 velocity=1 -> lower=0.523598775598 upper=5.75958653158 effort=2000 velocity=0.63
- joint j2s7s300_joint_3: limit lower=-174.532925 upper=174.532925 effort=2000 velocity=1 -> lower=-174.532925 upper=174.532925 effort=2000 velocity=0.63
- joint j2s7s300_joint_4: limit lower=0.523598775598 upper=5.75958653158 effort=2000 velocity=1 -> lower=0.523598775598 upper=5.75958653158 effort=2000 velocity=0.63
- joint j2s7s300_joint_5: limit lower=-174.532925 upper=174.532925 effort=2000 velocity=1 -> lower=-174.532925 upper=174.532925 effort=2000 velocity=0.85
- joint j2s7s300_joint_6: limit lower=0.523598775598 upper=5.75958653158 effort=2000 velocity=1 -> lower=0.523598775598 upper=5.75958653158 effort=2000 velocity=0.85
- joint j2s7s300_joint_7: limit lower=-174.532925 upper=174.532925 effort=2000 velocity=1 -> lower=-174.532925 upper=174.532925 effort=2000 velocity=0.85

File: multibody/parsing/test/sdf_parser_test/interface_api_test/arm.urdf (robot description, URDF)
Before this commit: robot arm, 2 links, 1 joints
Links:
- link L1: geometry collision sphere radius=0.4
- link L2: geometry collision sphere radius=0.4
